File: Archivos KiCAD/Green_Card.kicad_sch (KiCad schematic)
At the start: 0 parts

Commit message: Green Card casi completo
Parts:
- added BZ1: CEM-1203(42), symbol MicroProject-2026:Buzzer_Magnetico
- added C11, C12, C13, C17: 100nF, symbol MicroProject-2026:C
- added C14, C15, C16: 1uF, symbol MicroProject-2026:C_Tantalio
- added D10, D3, D4, D5, D6, D7, D8, D9: Rojo 5mm, symbol MicroProject-2026:LED
- added D11: RGB ánodo común, symbol MicroProject-2026:LED_RGB_CA
- added D12: 1N4148, symbol MicroProject-2026:Diodo
- added DS1: LTC-4627JR, symbol MicroProject-2026:LTC-4627JR
- added J2: DAC_OUT, symbol MicroProject-2026:Conn_01x02
- added JP1: Backlight, symbol MicroProject-2026:Jumper_2
- added LCD1: Nokia 5110 (LCD-10168), symbol MicroProject-2026:Nokia5110_LCD-10168
- added Q1, Q2, Q3, Q4: 2N3906, symbol MicroProject-2026:Q_PNP_2N3906
- added Q5, Q6, Q7, Q8: 2N3904, symbol MicroProject-2026:Q_NPN_2N3904
- added R10, R11, R12, R13: 330, symbol MicroProject-2026:R
- added R14, R15, R16, R17: 10k, symbol MicroProject-2026:R
- added R18, R19, R2, R20, R21, R3, R4, R5, R6, R7, R8, R9: 1k, symbol MicroProject-2026:R
- added R22: 180, symbol MicroProject-2026:R
- added R23, R24, R27: 100, symbol MicroProject-2026:R
- added R25, R26: 4.7k, symbol MicroProject-2026:R
- added RN1, RN2: 100, symbol MicroProject-2026:R_Network08_Isolated
- added RN3: 10k (común), symbol MicroProject-2026:R_Network15_Bussed
- added RV1: 10k lineal, symbol MicroProject-2026:R_Pot
- added SW2, SW3, SW4, SW5, SW6, SW7, SW8, SW9: SPDT, symbol MicroProject-2026:SW_SPDT
- added U101: NUCLEO-G431KB (copia de U1), symbol MicroProject-2026:NUCLEO-G431KB
- added U5, U6: MCP23017-E/SP, symbol MicroProject-2026:MCP23017_DIP28
Connections:
- new net: R5.1, SW5.2
- new net: R5.2, U5.4 (GPB3)
- new net: R9.1, SW9.2
- new net: Q1.2 (B), R10.2, R14.2
- new net: Q6.3 (C), R23.2
- new net: DS1.13 (C), RN2.14
- new net: RN2.3, U6.23 (GPA2)
- new net: R7.1, SW7.2
- new net: R7.2, U5.6 (GPB5)
- new net: D11.1 (R), R22.1
- new net: D11.3 (G), R23.1
- new net: D11.4 (B), R24.1
- new net: Q7.3 (C), R24.2
- new net: RN2.1, U6.21 (GPA0)
- new net: RN2.2, U6.22 (GPA1)
- new net: RN2.4, U6.24 (GPA3)
- new net: RN2.5, U6.25 (GPA4)
- new net: RN2.6, U6.26 (GPA5)
- new net: RN2.7, U6.27 (GPA6)
- new net: LCD1.8 (LED), R27.2
- new net: D7.1 (K), RN1.12
- new net: RN1.5, U5.25 (GPA4)
- new net: DS1.11 (F), RN2.11
- new net: DS1.14 (A), RN2.16
- new net: DS1.15 (G), RN2.10
- new net: DS1.16 (B), RN2.15
- new net: DS1.3 (D), RN2.13
- new net: DS1.5 (E), RN2.12
- new net: JP1.2, R27.1
- new net: Q4.2 (B), R13.2, R17.2
- new net: Q2.2 (B), R11.2, R15.2
- new net: R9.2, U5.8 (GPB7)
- new net: RN1.8, U5.28 (GPA7)
- new net: D10.1 (K), RN1.9
- new net: BZ1.2 (-), D12.2 (A), Q8.3 (C)
- new net: D4.1 (K), RN1.15
- new net: R6.1, SW6.2
- new net: R6.2, U5.5 (GPB4)
- new net: R3.1, SW3.2
- new net: R3.2, U5.2 (GPB1)
- new net: D9.1 (K), RN1.10
- new net: Q3.2 (B), R12.2, R16.2
- new net: R4.1, SW4.2
- new net: D6.1 (K), RN1.13
- new net: D5.1 (K), RN1.14
- new net: RN1.3, U5.23 (GPA2)
- new net: RN1.7, U5.27 (GPA6)
- new net: R8.1, SW8.2
- new net: D8.1 (K), RN1.11
- new net: Q5.3 (C), R22.2
- new net: R2.1, SW2.2
- new net: R2.2, U5.1 (GPB0)
- new net: R8.2, U5.7 (GPB6)
- new net: D3.1 (K), RN1.16
- new net: RN1.6, U5.26 (GPA5)
- new net: RN1.1, U5.21 (GPA0)
- new net: R4.2, U5.3 (GPB2)
- new net: RN1.2, U5.22 (GPA1)
- new net: RN1.4, U5.24 (GPA3)
- new net +3V3_IO: C11.1, C12.1, C14.1 (+), C15.1 (+), D10.2 (A), D3.2 (A), D4.2 (A), D5.2 (A), D6.2 (A), D7.2 (A), D8.2 (A), D9.2 (A), Q1.1 (E), Q2.1 (E), Q3.1 (E), Q4.1 (E), R14.1, R15.1, R16.1, R17.1, R25.1, R26.1, SW2.1, SW3.1, SW4.1, SW5.1, SW6.1, SW7.1, SW8.1, SW9.1, U5.9 (VDD), U6.15 (A0), U6.9 (VDD)
- new net +3V3_LCD: C13.1, C16.1 (+), JP1.1, LCD1.1 (VCC)
- new net +5V_EXT: BZ1.1 (+), D11.2 (A), D12.1 (K)
- new net ARC_RES1(U6_GPA7): U6.28 (GPA7)
- new net ARC_RES2(U6_GPB4): U6.5 (GPB4)
- new net ARC_RES3(U6_GPB5): U6.6 (GPB5)
- new net ARC_RES4(U6_GPB6): U6.7 (GPB6)
- new net ARC_RES5(U6_GPB7): U6.8 (GPB7)
- new net AVDD: RV1.1, U101.CN3-13 (AREF/AVDD)
- new net BUZZER(PB6): R21.1, U101.CN4-9 (D6/PB6)
- new net DAC_OUT(PA4): J2.1 (Pin_1), U101.CN3-9 (A3/PA4)
- new net DIG1: DS1.1 (DIG1), Q1.3 (C)
- new net DIG1_SEL: R10.1, U6.1 (GPB0)
- new net DIG2: DS1.2 (DIG2), Q2.3 (C)
- new net DIG2_SEL: R11.1, U6.2 (GPB1)
- new net DIG3: DS1.6 (DIG3), Q3.3 (C)
- new net DIG3_SEL: R12.1, U6.3 (GPB2)
- new net DIG4: DS1.8 (DIG4), Q4.3 (C)
- new net DIG4_SEL: R13.1, U6.4 (GPB3)
- new net GND: C11.2, C12.2, C13.2, C14.2 (-), C15.2 (-), C16.2 (-), C17.2, J2.2 (Pin_2), LCD1.2 (GND), Q5.1 (E), Q6.1 (E), Q7.1 (E), Q8.1 (E), RN3.16 (COM), RV1.3, SW2.3, SW3.3, SW4.3, SW5.3, SW6.3, SW7.3, SW8.3, SW9.3, U101.CN3-2 (GND), U101.CN4-4 (GND), U5.10 (VSS), U5.15 (A0), U5.16 (A1), U5.17 (A2), U6.10 (VSS), U6.16 (A1), U6.17 (A2)
- new net I2C1_SCL(PA15): R25.2, U101.CN3-7 (A5/PA6+PA15), U5.12 (SCL), U6.12 (SCL)
- new net I2C1_SDA(PB7): R26.2, U101.CN3-8 (A4/PA5+PB7), U5.13 (SDA), U6.13 (SDA)
- new net LCD_CE(PA11): LCD1.3 (SCE), U101.CN4-13 (D10/PA11)
- new net LCD_DC(PA12): LCD1.5 (D/C), U101.CN4-5 (D2/PA12)
- new net NRST: LCD1.4 (RST), U101.CN3-3 (NRST), U101.CN4-3 (NRST), U5.18 (RESET), U6.18 (RESET)
- new net PD_BUZZER: Q8.2 (B), R21.2, RN3.4
- new net PD_RGB_B: Q7.2 (B), R20.2, RN3.3
- new net PD_RGB_G: Q6.2 (B), R19.2, RN3.2
- new net PD_RGB_R: Q5.2 (B), R18.2, RN3.1
- new net POT(PA0): C17.1, RV1.2, U101.CN3-12 (A0/PA0)
- new net RES_ARCADE(PA1): U101.CN3-11 (A1/PA1)
- new net RES_ARCADE(PA8): U101.CN4-12 (D9/PA8)
- new net RES_FTDI_RX(PA10): U101.CN4-2 (D0/PA10)
- new net RES_FTDI_TX(PA9): U101.CN4-1 (D1/PA9)
- new net RGB_B(PB0): R20.1, U101.CN4-6 (D3/PB0)
- new net RGB_G(PA7): R19.1, U101.CN3-6 (A6/PA7)
- new net RGB_R(PB4): R18.1, U101.CN4-15 (D12/PB4)
- new net SPI1_MOSI(PB5): LCD1.6 (DN(MOSI)), U101.CN4-14 (D11/PB5)
- new net SPI1_SCK(PB3): LCD1.7 (SCLK), U101.CN3-15 (D13/PB3)
- no-connect marks 0 -> 26
Other:
- note added: "ANALÓGICO: potenciómetro (ADC) y salida del DAC"
- note added: "C11/C14: desacople de U5, junto a los pines 9 (VDD) y 10 (VSS). Dirección: A2 A1 A0 = 000 -> 0x20 (0100 A2 A1 A0, DS20001952E). LED encendido = GPAx en 0 (U5 absorbe la corriente). Switch hacia +3V3_IO = 1, hacia GND = 0. R2-R9 (1k) limitan a 3.3 mA si un pin de GPB se configura como salida por error."
- note added: "D11: COM-10821, ánodo a +5V_EXT. VF: R 2.0 V, G/B 3.2 V; IF máx 20 mA. Pata más larga = ánodo; el orden R-A-G-B varía según el lote: verificar con multímetro antes de cablear. Q5-Q8 (2N3904, 1=E 2=B 3=C): base con 1k desde el MCU; RN3 mantiene apagados los transistores mientras los pines del MCU están en alta impedancia (tras un reset). BZ1: transductor magnético de excitación externa (3.0-5.0 Vo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"
- note added: "GREEN_CARD - Conexiones de todos los comandos verdes"
- note added: "IMPORTANTE: el LTC-4627JR es de ÁNODO común (datasheet Lite-On DS30-2000-185 y DigiKey), aunque la lista de materiales lo describe como cátodo común Y no estoy seguro de cual tenemos realmente. Por eso los dígitos usan PNP (comprar 4 x 2N3906). U6: A2 A1 A0 = 001 -> 0x21. C12/C15: desacople junto a los pines 9 y 10. ARC_RES1-5: pines de U6 reservados para el teclado del Arcade."
- note added: "IN0"
- note added: "IN1"
- note added: "IN2"
- note added: "IN3"
- note added: "IN4"
- note added: "IN5"
- note added: "IN6"
- note added: "IN7"
- note added: "J2: salida del DAC1_OUT1 (AOUT/VOUT) para multímetro u osciloscopio. Con buffer: carga >= 5 kOhm y <= 50 pF; salida de 0.2 V a VREF+ - 0.2 V (DS12589 5.3.19)."
- note added: "LCD Nokia 5110 (SPI1)"
- note added: "LCD1: SparkFun LCD-10168 (PCD8544). VCC 2.7-3.3 V y entradas de 3.6 V máx: se alimenta de +3V3_LCD. RST unido a NRST: la LCD se reinicia con el MCU y con SW1. PCD8544 8.1: RES debe estar en bajo cuando VDD llega a su mínimo; se cumple si se enciende primero la fuente externa (NRST queda en 0 con la Nucleo apagada). SCLK máx 4 MHz (PCD8544 12). SCE puede quedar en bajo entre bytes (PCD8544 8). Bac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"
- note added: "OUT0"
- note added: "OUT1"
- note added: "OUT2"
- note added: "OUT3"
- note added: "OUT4"
- note added: "OUT5"
- note added: "OUT6"
- note added: "OUT7"
- note added: "PWM: LED RGB (TIM3) y buzzer (TIM4)"
- note added: "Q1-Q4 (2N3906, PNP): conmutan el ánodo de cada dígito desde +3V3_IO. Dígito encendido = GPBx de U6 en 0. R14-R17 (10k) mantienen apagados los PNP mientras U6 está en reset (pines en alta impedancia). Segmento encendido = GPAx de U6 en 0 (U6 absorbe). RN2 limita la corriente; DP y dos puntos sin usar."
- note added: "R25/R26: pull-ups del bus I2C1 a +3V3_IO"
- note added: "RN2: red de 100 Ohm (DIP-16)"
- note added: "RV1 (COM-09806): extremos entre AVDD (CN3-13) y GND; el ADC queda ratiométrico y PA0 nunca supera VDDA (DS12589 5.2 Tabla 14). C17 (100 nF) junto a PA0: reserva de carga para el muestreo y filtro. PA0 = ADC12_IN1, canal rápido (DS12589 4.10 Tabla 12; 5.3.18 Tabla 61)."
- note added: "TARJETA - copia de U1 como guía de conexión (etiquetas FUNCION(PIN))"
- note added: "U101 = copia de U1 (hoja Setup_Seguridad), excluida de BOM y placa: solo guía de conexión. X = pin sin conexión (estado de cada pin en Setup_Seguridad). PA2/PA3 = USART2 al VCP."
- note added: "U5 MCP23017 #1 (0x20): 8 LEDs OUT0-7 y 8 switches IN0-7"
- note added: "U6 MCP23017 #2 (0x21): display LTC-4627JR de 4 dígitos (ÁNODO común) CAMBIAR DESPUÉS EN DADO CASO SEA CÁTODO"
- note removed: "GREEN_CARD - comandos verdes"
- note removed: "Hoja pendiente: se desarrollará después de Setup_Seguridad."
